File: workshop1/APC.sch (KiCad schematic (older format))
At the start: 16 parts, among them J1 Conn_01x02, SW1 SW_SPDT, U1 NE556

Commit message: Added footprints
Parts:
- BT1: footprint (none) -> Battery:BatteryHolder_Eagle_12BH611-GR
- C1, C2: footprint (none) -> Capacitor_SMD:C_0603_1608Metric_Pad1.05x0.95mm_HandSolder
- C3: footprint (none) -> Capacitor_SMD:CP_Elec_5x3
- J1: footprint (none) -> Connector_Wire:SolderWirePad_1x02_P7.62mm_Drill2.5mm
- R1: footprint (none) -> Resistor_SMD:R_0603_1608Metric_Pad1.05x0.95mm_HandSolder
- RV1, RV2, RV3: footprint (none) -> Potentiometer_THT:Potentiometer_Bourns_PTV09A-1_Single_Vertical
- SW1: footprint (none) -> Button_Switch_SMD:SW_SPDT_CK-JS102011SAQN
- TP1, TP2, TP3, TP4, TP5: footprint (none) -> TestPoint:TestPoint_Pad_D1.5mm
- U1: footprint (none) -> Package_SO:SOIC-14_3.9x8.7mm_P1.27mm
Connections:
- net +9V: now also TP1.1
- net at BT1.1 (+), SW1.2 (B): no longer TP1.1
Other:
- moved on the sheet: TP1

Commit message: Slight changes to the schematic
Parts:
- added H1, H2, H3, H4: MountingHole, symbol Mechanical:MountingHole
Connections:
- wire segments 50 -> 51
Other:
- moved on the sheet: RV1, RV2
Changed lines of the file:
@@
 EESchema Schematic File Version 4
-LIBS:APC-cache
-EELAYER 30 0
+EELAYER 29 0
 EELAYER END
 $Descr A4 11693 8268
@@
 Connection ~ 7750 3250
 Wire Wire Line
-	8100 3250 7750 3250
-NoConn ~ 8100 3650
-Wire Wire Line
-	8450 3500 8250 3500
+	8400 3250 7750 3250
+NoConn ~ 8400 3650
+Wire Wire Line
+	8100 3500 8250 3500
 $Comp
 L power:+9V #PWR0111
 U 1 1 5D838B33
-P 8450 3500
-F 0 "#PWR0111" H 8450 3350 50  0001 C CNN
-F 1 "+9V" V 8465 3628 50  0000 L CNN
-F 2 "" H 8450 3500 50  0001 C CNN
-F 3 "" H 8450 3500 50  0001 C CNN
-	1    8450 3500
-	0    1    1    0
-$EndComp
-Wire Wire Line
-	8100 3350 8100 3250
+P 8100 3500
+F 0 "#PWR0111" H 8100 3350 50  0001 C CNN
+F 1 "+9V" V 8115 3628 50  0000 L CNN
+F 2 "" H 8100 3500 50  0001 C CNN
+F 3 "" H 8100 3500 50  0001 C CNN
+	1    8100 3500
+	0    -1   -1   0
+$EndComp
+Wire Wire Line
+	8400 3350 8400 3250
 $Comp
 L Device:R_POT RV2
 U 1 1 5D803438
-P 8100 3500
-F 0 "RV2" H 8030 3546 50  0000 R CNN
-F 1 "1M" H 8030 3455 50  0000 R CNN
-F 2 "Potentiometer_THT:Potentiometer_Bourns_PTV09A-1_Single_Vertical" H 8100 3500 50  0001 C CNN
-F 3 "~" H 8100 3500 50  0001 C CNN
-	1    8100 3500
-	1    0    0    -1
+P 8400 3500
+F 0 "RV2" H 8330 3546 50  0000 R CNN
+F 1 "1M" H 8330 3455 50  0000 R CNN
+F 2 "Potentiometer_THT:Potentiometer_Bourns_PTV09A-1_Single_Vertical" H 8400 3500 50  0001 C CNN
+F 3 "~" H 8400 3500 50  0001 C CNN
+	1    8400 3500
+	-1   0    0    1
 $EndComp
 $Comp
@@
 $EndComp
 Wire Wire Line
-	8850 3250 8100 3250
-Connection ~ 8100 3250
+	8850 3250 8400 3250
+Connection ~ 8400 3250
 $Comp
 L Connector:TestPoint TP4
@@
 $EndComp
 $Comp
+L power:+9V #PWR0109
+U 1 1 5D81EBEF
+P 6350 3000
+F 0 "#PWR0109" H 6350 2850 50  0001 C CNN
+F 1 "+9V" V 6365 3128 50  0000 L CNN
+F 2 "" H 6350 3000 50  0001 C CNN
+F 3 "" H 6350 3000 50  0001 C CNN
+	1    6350 3000
+	0    1    1    0
+$EndComp
+NoConn ~ 6100 2850
+Wire Wire Line
+	3050 2650 3300 2650
+$Comp
 L Device:R_POT RV1
 U 1 1 5D80479C
@@
 F 3 "~" H 6100 3000 50  0001 C CNN
 	1    6100 3000
-	-1   0    0    1
-$EndComp
-$Comp
-L power:+9V #PWR0109
-U 1 1 5D81EBEF
-P 5900 3000
-F 0 "#PWR0109" H 5900 2850 50  0001 C CNN
-F 1 "+9V" V 5915 3128 50  0000 L CNN
-F 2 "" H 5900 3000 50  0001 C CNN
-F 3 "" H 5900 3000 50  0001 C CNN
-	1    5900 3000
-	0    -1   -1   0
-$EndComp
-NoConn ~ 6100 2850
-Wire Wire Line
-	3050 2650 3300 2650
+	1    0    0    -1
+$EndComp
+Wire Wire Line
+	6350 3000 6250 3000
+$Comp
+L Mechanical:MountingHole H2
+U 1 1 5D82A873
+P 8400 5950
+F 0 "H2" H 8500 5996 50  0000 L CNN
+F 1 "MountingHole" H 8500 5905 50  0000 L CNN
+F 2 "" H 8400 5950 50  0001 C CNN
+F 3 "~" H 8400 5950 50  0001 C CNN
+	1    8400 5950
+	1    0    0    -1
+$EndComp
+$Comp
+L Mechanical:MountingHole H3
+U 1 1 5D82B570
+P 9250 5950
+F 0 "H3" H 9350 5996 50  0000 L CNN
+F 1 "MountingHole" H 9350 5905 50  0000 L CNN
+F 2 "" H 9250 5950 50  0001 C CNN
+F 3 "~" H 9250 5950 50  0001 C CNN
+	1    9250 5950
+	1    0    0    -1
+$EndComp
+$Comp
+L Mechanical:MountingHole H4
+U 1 1 5D82B8FB
+P 10000 5950
+F 0 "H4" H 10100 5996 50  0000 L CNN
+F 1 "MountingHole" H 10100 5905 50  0000 L CNN
+F 2 "" H 10000 5950 50  0001 C CNN
+F 3 "~" H 10000 5950 50  0001 C CNN
+	1    10000 5950
+	1    0    0    -1
+$EndComp
+$Comp
+L Mechanical:MountingHole H1
+U 1 1 5D82BC64
+P 7650 5950
+F 0 "H1" H 7750 5996 50  0000 L CNN
+F 1 "MountingHole" H 7750 5905 50  0000 L CNN
+F 2 "" H 7650 5950 50  0001 C CNN
+F 3 "~" H 7650 5950 50  0001 C CNN
+	1    7650 5950
+	1    0    0    -1
+$EndComp
 $EndSCHEMATC
