File: KiCAD_Projektdateien/workshop_teil1/APC.sch (KiCad schematic (older format))
At the start: 20 parts, among them J1 Conn_01x02, SW1 SW_SPDT, U1 NE556

Commit message: Added footprints for mounting holes
Parts:
- H1, H2, H3, H4: footprint (none) -> MountingHole:MountingHole_3.2mm_M3
Changed lines of the file:
@@
 EESchema Schematic File Version 4
-EELAYER 29 0
+LIBS:APC-cache
+EELAYER 30 0
 EELAYER END
 $Descr A4 11693 8268
@@
 F 0 "H2" H 8500 5996 50  0000 L CNN
 F 1 "MountingHole" H 8500 5905 50  0000 L CNN
-F 2 "" H 8400 5950 50  0001 C CNN
+F 2 "MountingHole:MountingHole_3.2mm_M3" H 8400 5950 50  0001 C CNN
 F 3 "~" H 8400 5950 50  0001 C CNN
 	1    8400 5950
@@
 F 0 "H3" H 9350 5996 50  0000 L CNN
 F 1 "MountingHole" H 9350 5905 50  0000 L CNN
-F 2 "" H 9250 5950 50  0001 C CNN
+F 2 "MountingHole:MountingHole_3.2mm_M3" H 9250 5950 50  0001 C CNN
 F 3 "~" H 9250 5950 50  0001 C CNN
 	1    9250 5950
@@
 F 0 "H4" H 10100 5996 50  0000 L CNN
 F 1 "MountingHole" H 10100 5905 50  0000 L CNN
-F 2 "" H 10000 5950 50  0001 C CNN
+F 2 "MountingHole:MountingHole_3.2mm_M3" H 10000 5950 50  0001 C CNN
 F 3 "~" H 10000 5950 50  0001 C CNN
 	1    10000 5950
@@
 F 0 "H1" H 7750 5996 50  0000 L CNN
 F 1 "MountingHole" H 7750 5905 50  0000 L CNN
-F 2 "" H 7650 5950 50  0001 C CNN
+F 2 "MountingHole:MountingHole_3.2mm_M3" H 7650 5950 50  0001 C CNN
 F 3 "~" H 7650 5950 50  0001 C CNN
 	1    7650 5950
