File: KiCAD_Projektdateien/workshop_teil2/APC.sch (KiCad schematic (older format))
At the start: 20 parts, among them J1 Conn_01x02, SW1 SW_SPDT, U1 NE556

Commit message: created another BOM
Parts:
- C1: Distributor (none) -> Mouser; Manufacturer (none) -> Vishay / Vitramon; Order Number (none) -> 77-VJ0603V103ZXJPBC; Part Number (none) -> VJ0603V103ZXJPW1BC
Changed lines of the file:
@@
 F 2 "Capacitor_SMD:C_0603_1608Metric_Pad1.05x0.95mm_HandSolder" H 5388 3750 50  0001 C CNN
 F 3 "~" H 5350 3900 50  0001 C CNN
+F 4 "Mouser" H 5350 3900 50  0001 C CNN "Distributor"
+F 5 "Vishay / Vitramon" H 5350 3900 50  0001 C CNN "Manufacturer"
+F 6 "77-VJ0603V103ZXJPBC" H 5350 3900 50  0001 C CNN "Order Number"
+F 7 "VJ0603V103ZXJPW1BC" H 5350 3900 50  0001 C CNN "Part Number"
 	1    5350 3900
 	0    -1   -1   0
